File: transistor-tester.kicad_pcb (KiCad board)
At the start: 2 copper layers, 77.3 x 90.6 mm, 19 parts, among them J1 Screw_Terminal_01x02, J2 NMOS Socket, J3 PMOS Socket, J4 NPN Socket, J5 PNP Socket, SW1 PMOS SW, SW2 NMOS SW

Commit message: latest
Routing:
- net PWR: track 0.00 -> 158.7 mm
- net LEDhi: track 0.00 -> 84.6 mm
- net Vlo: track 0.00 -> 54.2 mm
- net Net-(D1-K): track 0.00 -> 52.0 mm
- net Vhi: track 0.00 -> 49.2 mm
- net Net-(D2-K): track 0.00 -> 37.8 mm
- net LEDlo: track 0.00 -> 34.1 mm
- net Net-(R2-Pad2): track 0.00 -> 31.0 mm
- net Net-(J5-Pin_2): track 0.00 -> 25.3 mm

Commit message: Added product links to all kicad datasheet entries
Parts:
- D1, D2: value E-101 -> E-301
Changed lines of the file:
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@@
 			)
 		)
-		(property "Description" "Socket Terminal for TO-220 push-connect"
+		(property "Description" "Generic screw terminal, single row, 01x03, script generated (kicad-library-utils/schlib/autogen/connector/)"
 			(at 0 0 0)
 			(layer "F.Fab")
@@
 		)
 		(property ki_fp_filters "TerminalBlock*:*")
-		(sheetname "Root")
+		(sheetname "/")
 		(sheetfile "transistor-tester.kicad_sch")
 		(attr through_hole)
@@
 		)
 		(property ki_fp_filters "R_*")
-		(sheetname "Root")
+		(sheetname "/")
 		(sheetfile "transistor-tester.kicad_sch")
 		(attr through_hole)
@@
 			)
 		)
-		(property "Datasheet" "https://www.amazon.com/dp/B07H5G7GC6?ref_=ppx_hzsearch_conn_dt_b_fed_asin_title_4"
+		(property "Datasheet" "https://www.amazon.com/dp/B09ZTFKYCK?ref_=ppx_hzsearch_conn_dt_b_fed_asin_title_2&th=1"
 			(at 0 0 0)
 			(layer "F.Fab")
@@
 		)
 		(property ki_fp_filters "TerminalBlock*:*")
-		(sheetname "Root")
+		(sheetname "/")
 		(sheetfile "transistor-tester.kicad_sch")
 		(attr through_hole)
@@
 		)
 		(property ki_fp_filters "R_*")
-		(sheetname "Root")
+		(sheetname "/")
 		(sheetfile "transistor-tester.kicad_sch")
 		(attr through_hole)
@@
 			)
 		)
-		(property "Description" "Socket Terminal for TO-220 push-connect"
+		(property "Description" "Generic screw terminal, single row, 01x03, script generated (kicad-library-utils/schlib/autogen/connector/)"
 			(at 0 0 0)
 			(layer "F.Fab")
@@
 		)
 		(property ki_fp_filters "TerminalBlock*:*")
-		(sheetname "Root")
+		(sheetname "/")
 		(sheetfile "transistor-tester.kicad_sch")
 		(attr through_hole)
@@
 			)
 		)
-		(property "Value" "E-101"
+		(property "Value" "E-301"
 			(at 5.08 -0.73 90)
 			(layer "B.SilkS")
@@
 			)
 		)
-		(property "Datasheet" ""
+		(property "Datasheet" "https://www.mouser.com/ProductDetail/Semitec/E-301?qs=wgO0AD0o1vvnCxICGY3ceQ%3D%3D"
 			(at 0 0 270)
 			(unlocked yes)
@@
 		)
 		(property ki_fp_filters "TO-???* D_*")
-		(sheetname "Root")
+		(sheetname "/")
 		(sheetfile "transistor-tester.kicad_sch")
 		(attr through_hole)
@@
 			)
 		)
-		(property "Description" "Socket Terminal for TO-220 push-connect"
+		(property "Description" "Generic screw terminal, single row, 01x03, script generated (kicad-library-utils/schlib/autogen/connector/)"
 			(at 0 0 0)
 			(layer "F.Fab")
@@
 		)
 		(property ki_fp_filters "TerminalBlock*:*")
-		(sheetname "Root")
+		(sheetname "/")
 		(sheetfile "transistor-tester.kicad_sch")
 		(attr through_hole)
@@
 			)
 		)
-		(property "Datasheet" ""
+		(property "Datasheet" "https://www.amazon.com/dp/B073QMYKDM?ref_=ppx_hzsearch_conn_dt_b_fed_asin_title_10"
 			(at 0 0 0)
 			(layer "F.Fab")
@@
 		)
 		(property ki_fp_filters "LED* LED_SMD:* LED_THT:*")
-		(sheetname "Root")
+		(sheetname "/")
 		(sheetfile "transistor-tester.kicad_sch")
 		(attr through_hole)
@@
 			)
 		)
-		(property "Datasheet" "https://www.amazon.com/dp/B0CNLNTN5J?ref=ppx_yo2ov_dt_b_fed_asin_title&th=1"
+		(property "Datasheet" "https://www.amazon.com/dp/B08R9P9DFC?ref_=ppx_hzsearch_conn_dt_b_fed_asin_title_1&th=1"
 			(at 0 0 180)
 			(unlocked yes)
@@
 			)
 		)
-		(sheetname "Root")
+		(sheetname "/")
 		(sheetfile "transistor-tester.kicad_sch")
 		(pad "" np_thru_hole circle
@@
 			)
 		)
-		(property "Value" "E-101"
+		(property "Value" "E-301"
 			(at 5.08 0.87 90)
 			(layer "B.SilkS")
@@
 			)
 		)
-		(property "Datasheet" ""
+		(property "Datasheet" "https://www.mouser.com/ProductDetail/Semitec/E-301?qs=wgO0AD0o1vvnCxICGY3ceQ%3D%3D"
 			(at 0 0 90)
 			(unlocked yes)
@@
 		)
 		(property ki_fp_filters "TO-???* D_*")
-		(sheetname "Root")
+		(sheetname "/")
 		(sheetfile "transistor-tester.kicad_sch")
 		(attr through_hole)
@@
 		)
 		(property ki_fp_filters "R_*")
-		(sheetname "Root")
+		(sheetname "/")
 		(sheetfile "transistor-tester.kicad_sch")
 		(attr through_hole)
@@
 		)
 		(property ki_fp_filters "R_*")
-		(sheetname "Root")
+		(sheetname "/")
 		(sheetfile "transistor-tester.kicad_sch")
 		(attr through_hole)
@@
 			)
 		)
-		(property "Datasheet" ""
+		(property "Datasheet" "https://www.amazon.com/dp/B073QMYKDM?ref_=ppx_hzsearch_conn_dt_b_fed_asin_title_10"
 			(at 0 0 0)
 			(layer "F.Fab")
@@
 		)
 		(property ki_fp_filters "LED* LED_SMD:* LED_THT:*")
-		(sheetname "Root")
+		(sheetname "/")
 		(sheetfile "transistor-tester.kicad_sch")
 		(attr through_hole)
@@
 			)
 		)
-		(property "Description" "Socket Terminal for TO-220 push-connect"
+		(property "Description" "Generic screw terminal, single row, 01x03, script generated (kicad-library-utils/schlib/autogen/connector/)"
 			(at 0 0 0)
 			(layer "F.Fab")
@@
 		)
 		(property ki_fp_filters "TerminalBlock*:*")
-		(sheetname "Root")
+		(sheetname "/")
 		(sheetfile "transistor-tester.kicad_sch")
 		(attr through_hole)
@@
 			)
 		)
-		(property "Datasheet" ""
+		(property "Datasheet" "https://www.amazon.com/dp/B08R9P9DFC?ref_=ppx_hzsearch_conn_dt_b_fed_asin_title_1&th=1"
 			(at 0 0 0)
 			(unlocked yes)
@@
 			)
 		)
-		(sheetname "Root")
+		(sheetname "/")
 		(sheetfile "transistor-tester.kicad_sch")
 		(pad "" np_thru_hole circle
